File: day-star.kicad_pcb (KiCad board)
At the start: 2 copper layers, 119.3 x 41.8 mm, 34 parts, among them P1 PWR_CONN, Q1 Q_PMOS_DGS, Q2 Q_NMOS_DGS, Q3 Q_NMOS_DGS, U1 LM311N

Commit message: Continuing shiggles
Parts:
- removed the D1 at (105.0, 27.0)
- removed the D1 at (65.0, 27.0)
- removed the D1 at (25.0, 27.0)
- removed the Q1 at (105.0, 33.2)
- removed the Q1 at (65.0, 33.2)
- removed the Q2 at (109.6, 29.0)
- removed the Q2 at (69.6, 29.0)
- removed the Q3 at (113.1, 29.0)
- removed the Q3 at (73.1, 29.0)
- removed the R4 at (108.0, 34.1)
- removed the R4 at (68.0, 34.1)
- removed the R5 at (110.6, 34.1)
- removed the R5 at (70.6, 34.1)
- removed the R6 at (112.1, 32.5)
- removed the R6 at (72.1, 32.5)
- removed the R7 at (105.0, 22.9)
- removed the R7 at (65.0, 22.9)
- removed the U1 at (114.6, 36.1)
- removed the U1 at (74.6, 36.1)
- added D1: LED, Terminal_Blocks:TerminalBlock_Pheonix_MKDS1.5-2pol, F.Cu at (35.9, 20.7)
- added D2: LED, Terminal_Blocks:TerminalBlock_Pheonix_MKDS1.5-2pol, F.Cu at (81.8, 50.7)
- added D3: LED, Terminal_Blocks:TerminalBlock_Pheonix_MKDS1.5-2pol, F.Cu at (90.0, 77.7)
- added Q4: Q_PMOS_DGS, TO_SOT_Packages_THT:TO-220_Neutral123_Horizontal_LargePads, B.Cu at (73.2, 51.1)
- added Q5: Q_NMOS_DGS, agg:SOT-23, F.Cu at (94.1, 30.7)
- added Q6: Q_NMOS_DGS, agg:SOT-23, F.Cu at (83.9, 30.7)
- added Q7: Q_PMOS_DGS, TO_SOT_Packages_THT:TO-220_Neutral123_Horizontal_LargePads, B.Cu at (73.2, 84.3)
- added Q8: Q_NMOS_DGS, agg:SOT-23, F.Cu at (94.1, 63.9)
- added Q9: Q_NMOS_DGS, agg:SOT-23, F.Cu at (83.9, 63.9)
- added R1: 2k, agg:0603, F.Cu at (39.4, 51.9)
- added R10: 2k2, agg:0603, F.Cu at (102.5, 29.1)
- added R11: 0R03, Resistors_SMD:R_2512, B.Cu at (82.9, 38.3)
- added R12: 1k, agg:0603, F.Cu at (81.9, 80.9)
- added R13: 1k, agg:0603, F.Cu at (102.5, 62.2)
- added R14: 2k2, agg:0603, F.Cu at (81.9, 77.4)
- added R15: 0R03, Resistors_SMD:R_2512, B.Cu at (82.9, 71.5)
- added R2: 1k, agg:0603, F.Cu at (36.3, 51.9)
- added R8: 1k, agg:0603, F.Cu at (81.9, 43.8)
- added R9: 1k, agg:0603, F.Cu at (81.9, 46.3)
- added U2: LM311N, agg:MSOP-8, F.Cu at (90.4, 37.7)
- added U3: LM311N, agg:MSOP-8, F.Cu at (90.4, 70.9)
- P1: footprint agg:SIL-254P-02 -> Terminal_Blocks:TerminalBlock_Pheonix_MKDS1.5-2pol
- R3: value 11K -> 11k9
- R7: value 0R3 -> 0R03; footprint Resistors_ThroughHole:Resistor_Horizontal_RM25mm -> Resistors_SMD:R_2512
- RV1: value 1k -> 100R
- moved P1 40.6 mm to (22.3, 47.3)
- moved C1 34.7 mm to (37.8, 50.4)
- moved PWR1 34.7 mm to (38.9, 49.2)
- moved R3 34.7 mm to (47.5, 48.6)
- moved RV1 34.7 mm to (49.8, 48.0)
- moved C2 34.7 mm to (41.9, 50.4)
- moved C3 34.7 mm to (41.9, 45.5)
- moved R7 14.2 mm to (39.0, 25.1)
- moved Q1 0.72 mm to (24.8, 32.5)
Routing:
- net +36V: track 157.4 -> 62.5 mm
- net GND: track 31.8 -> 117.7 mm, vias 9 -> 3
- net /DriveA/VREF: track 99.0 -> 20.5 mm, vias 6 -> 0
- net +12V: track 100.5 -> 22.2 mm, vias 4 -> 0
- net /DriveA/SENSE: track 67.9 -> 16.1 mm
- net Net-(D1-Pad2): track 36.1 -> 17.8 mm
- net Net-(Q3-Pad2): track 22.6 -> 7.53 mm
- net Net-(Q1-Pad2): track 20.3 -> 7.32 mm
- net Net-(Q2-Pad2): track 14.0 -> 4.67 mm
- net Net-(C1-Pad1): track 1.38 -> 4.68 mm
- net Net-(Q3-Pad1): track 4.71 -> 1.57 mm
- added copper zone on B.Cu, net /DriveA/SENSE
Other:
- board size 119.3 x 41.8 mm -> 37.5 x 40 mm
- net class 3A added: clearance 0.5, trace_width 2, via_dia 0.6, via_drill 0.4
