File: drive.sch (KiCad schematic (older format))
At the start: 9 parts, among them Q1 Q_PMOS_DGS, Q2 Q_NMOS_DGS, Q3 Q_NMOS_DGS, U1 LM311N

Commit message: Continuing shiggles
Parts:
- D1: footprint agg:SIL-254P-02 -> Terminal_Blocks:TerminalBlock_Pheonix_MKDS1.5-2pol
- R7: value 0R3 -> 0R03; footprint Resistors_ThroughHole:Resistor_Horizontal_RM25mm -> Resistors_SMD:R_2512
Connections:
- net +36V: no longer Q1.3 (S)
- net GND: no longer R7.2
- new net GNDPWR: R7.2
- new net VPP: Q1.3 (S)
Changed lines of the file:
@@
 AR Path="/57724CA7/57724742" Ref="Q5"  Part="1"
 AR Path="/57724D0D/57724742" Ref="Q8"  Part="1"
-F 0 "Q8" H 2350 1400 50  0001 R CNN
+F 0 "Q2" H 2350 1400 50  0001 R CNN
 F 1 "Q_NMOS_DGS" V 2300 1300 50  0001 R CNN
 F 2 "agg:SOT-23" H 2250 1450 50  0001 C CNN
@@
 AR Path="/57724CA7/57724748" Ref="R9"  Part="1"
 AR Path="/57724D0D/57724748" Ref="R13"  Part="1"
-F 0 "R13" V 1930 1200 50  0001 C CNN
+F 0 "R5" V 1930 1200 50  0001 C CNN
 F 1 "1k" V 1850 1200 50  0000 C CNN
 F 2 "agg:0603" V 1780 1200 50  0001 C CNN
@@
 AR Path="/57724CA7/5772474E" Ref="R10"  Part="1"
 AR Path="/57724D0D/5772474E" Ref="R14"  Part="1"
-F 0 "R14" V 1930 1500 50  0001 C CNN
+F 0 "R6" V 1930 1500 50  0001 C CNN
 F 1 "2k2" V 1850 1500 50  0000 C CNN
 F 2 "agg:0603" V 1780 1500 50  0001 C CNN
@@
 AR Path="/57724CA7/57724755" Ref="D2"  Part="1"
 AR Path="/57724D0D/57724755" Ref="D3"  Part="1"
-F 0 "D3" H 2450 1650 50  0001 C CNN
+F 0 "D1" H 2450 1650 50  0001 C CNN
 F 1 "LED" H 2450 1450 50  0001 C CNN
-F 2 "agg:SIL-254P-02" H 2450 1550 50  0001 C CNN
+F 2 "Terminal_Blocks:TerminalBlock_Pheonix_MKDS1.5-2pol" H 2450 1550 50  0001 C CNN
 F 3 "" H 2450 1550 50  0000 C CNN
 	1    2450 1550
@@
 AR Path="/57724CA7/5772475B" Ref="R11"  Part="1"
 AR Path="/57724D0D/5772475B" Ref="R15"  Part="1"
-F 0 "R15" V 2530 1900 50  0001 C CNN
-F 1 "0R3" V 2450 1900 50  0000 C CNN
-F 2 "Resistors_ThroughHole:Resistor_Horizontal_RM25mm" V 2380 1900 50  0001 C CNN
-F 3 "" H 2450 1900 50  0000 C CNN
+F 0 "R7" V 2530 1900 50  0001 C CNN
+F 1 "0R03" V 2450 1900 50  0000 C CNN
+F 2 "Resistors_SMD:R_2512" V 2380 1900 50  0001 C CNN
+F 3 "http://www.farnell.com/datasheets/1518406.pdf" H 2450 1900 50  0001 C CNN
 	1    2450 1900
 	1    0    0    -1
@@
 Connection ~ 2450 1750
 $Comp
-L GND #PWR016
-U 1 1 57724765
-P 2450 2050
-AR Path="/577246EF/57724765" Ref="#PWR016"  Part="1"
-AR Path="/57724CA7/57724765" Ref="#PWR024"  Part="1"
-AR Path="/57724D0D/57724765" Ref="#PWR032"  Part="1"
-F 0 "#PWR032" H 2450 1800 50  0001 C CNN
-F 1 "GND" H 2450 1900 50  0000 C CNN
-F 2 "" H 2450 2050 50  0000 C CNN
-F 3 "" H 2450 2050 50  0000 C CNN
-	1    2450 2050
-	1    0    0    -1
-$EndComp
-$Comp
-L +36V #PWR017
+L +36V #PWR22
 U 1 1 5772476B
 P 2150 850
-AR Path="/577246EF/5772476B" Ref="#PWR017"  Part="1"
-AR Path="/57724CA7/5772476B" Ref="#PWR025"  Part="1"
-AR Path="/57724D0D/5772476B" Ref="#PWR033"  Part="1"
-F 0 "#PWR033" H 2150 700 50  0001 C CNN
+AR Path="/577246EF/5772476B" Ref="#PWR22"  Part="1"
+AR Path="/57724CA7/5772476B" Ref="#PWR30"  Part="1"
+AR Path="/57724D0D/5772476B" Ref="#PWR38"  Part="1"
+F 0 "#PWR22" H 2150 700 50  0001 C CNN
 F 1 "+36V" H 2150 990 50  0000 C CNN
 F 2 "" H 2150 850 50  0000 C CNN
@@
 AR Path="/57724CA7/57724771" Ref="Q4"  Part="1"
 AR Path="/57724D0D/57724771" Ref="Q7"  Part="1"
-F 0 "Q7" H 2650 1200 50  0001 R CNN
+F 0 "Q1" H 2650 1200 50  0001 R CNN
 F 1 "Q_PMOS_DGS" H 3000 1100 50  0001 R CNN
 F 2 "TO_SOT_Packages_THT:TO-220_Neutral123_Horizontal_LargePads" H 2550 1250 50  0001 C CNN
@@
 AR Path="/57724CA7/57724777" Ref="R8"  Part="1"
 AR Path="/57724D0D/57724777" Ref="R12"  Part="1"
-F 0 "R12" V 2230 1000 50  0001 C CNN
+F 0 "R4" V 2230 1000 50  0001 C CNN
 F 1 "1k" V 2150 1000 50  0000 C CNN
 F 2 "agg:0603" V 2080 1000 50  0001 C CNN
@@
 $EndComp
 $Comp
-L GND #PWR018
+L GND #PWR23
 U 1 1 5772477D
 P 2150 1550
-AR Path="/577246EF/5772477D" Ref="#PWR018"  Part="1"
-AR Path="/57724CA7/5772477D" Ref="#PWR026"  Part="1"
-AR Path="/57724D0D/5772477D" Ref="#PWR034"  Part="1"
-F 0 "#PWR034" H 2150 1300 50  0001 C CNN
+AR Path="/577246EF/5772477D" Ref="#PWR23"  Part="1"
+AR Path="/57724CA7/5772477D" Ref="#PWR31"  Part="1"
+AR Path="/57724D0D/5772477D" Ref="#PWR39"  Part="1"
+F 0 "#PWR23" H 2150 1300 50  0001 C CNN
 F 1 "GND" H 2150 1400 50  0000 C CNN
 F 2 "" H 2150 1550 50  0000 C CNN
@@
 AR Path="/57724CA7/57724783" Ref="Q6"  Part="1"
 AR Path="/57724D0D/57724783" Ref="Q9"  Part="1"
-F 0 "Q9" H 2050 1900 50  0001 R CNN
+F 0 "Q3" H 2050 1900 50  0001 R CNN
 F 1 "Q_NMOS_DGS" V 2000 1800 50  0001 R CNN
 F 2 "agg:SOT-23" H 1950 1950 50  0001 C CNN
@@
 Connection ~ 1850 1350
 $Comp
-L +36V #PWR019
+L +36V #PWR20
 U 1 1 5772478A
 P 1850 1050
-AR Path="/577246EF/5772478A" Ref="#PWR019"  Part="1"
-AR Path="/57724CA7/5772478A" Ref="#PWR027"  Part="1"
-AR Path="/57724D0D/5772478A" Ref="#PWR035"  Part="1"
-F 0 "#PWR035" H 1850 900 50  0001 C CNN
+AR Path="/577246EF/5772478A" Ref="#PWR20"  Part="1"
+AR Path="/57724CA7/5772478A" Ref="#PWR28"  Part="1"
+AR Path="/57724D0D/5772478A" Ref="#PWR36"  Part="1"
+F 0 "#PWR20" H 1850 900 50  0001 C CNN
 F 1 "+36V" H 1850 1190 50  0000 C CNN
 F 2 "" H 1850 1050 50  0000 C CNN
@@
 $EndComp
 $Comp
-L +36V #PWR020
-U 1 1 57724790
-P 2450 950
-AR Path="/577246EF/57724790" Ref="#PWR020"  Part="1"
-AR Path="/57724CA7/57724790" Ref="#PWR028"  Part="1"
-AR Path="/57724D0D/57724790" Ref="#PWR036"  Part="1"
-F 0 "#PWR036" H 2450 800 50  0001 C CNN
-F 1 "+36V" H 2450 1090 50  0000 C CNN
-F 2 "" H 2450 950 50  0000 C CNN
-F 3 "" H 2450 950 50  0000 C CNN
-	1    2450 950
-	-1   0    0    -1
-$EndComp
-$Comp
-L GND #PWR021
+L GND #PWR21
 U 1 1 57724796
 P 1850 2050
-AR Path="/577246EF/57724796" Ref="#PWR021"  Part="1"
-AR Path="/57724CA7/57724796" Ref="#PWR029"  Part="1"
-AR Path="/57724D0D/57724796" Ref="#PWR037"  Part="1"
-F 0 "#PWR037" H 1850 1800 50  0001 C CNN
+AR Path="/577246EF/57724796" Ref="#PWR21"  Part="1"
+AR Path="/57724CA7/57724796" Ref="#PWR29"  Part="1"
+AR Path="/57724D0D/57724796" Ref="#PWR37"  Part="1"
+F 0 "#PWR21" H 1850 1800 50  0001 C CNN
 F 1 "GND" H 1850 1900 50  0000 C CNN
 F 2 "" H 1850 2050 50  0000 C CNN
@@
 $EndComp
 $Comp
-L GND #PWR022
+L GND #PWR19
 U 1 1 577247B5
 P 1150 2150
-AR Path="/577246EF/577247B5" Ref="#PWR022"  Part="1"
-AR Path="/57724CA7/577247B5" Ref="#PWR030"  Part="1"
-AR Path="/57724D0D/577247B5" Ref="#PWR038"  Part="1"
-F 0 "#PWR038" H 1150 1900 50  0001 C CNN
+AR Path="/577246EF/577247B5" Ref="#PWR19"  Part="1"
+AR Path="/57724CA7/577247B5" Ref="#PWR27"  Part="1"
+AR Path="/57724D0D/577247B5" Ref="#PWR35"  Part="1"
+F 0 "#PWR19" H 1150 1900 50  0001 C CNN
 F 1 "GND" H 1150 2000 50  0000 C CNN
 F 2 "" H 1150 2150 50  0000 C CNN
@@
 $EndComp
 $Comp
-L +12V #PWR023
+L +12V #PWR18
 U 1 1 577247BB
 P 1150 1550
-AR Path="/577246EF/577247BB" Ref="#PWR023"  Part="1"
-AR Path="/57724CA7/577247BB" Ref="#PWR031"  Part="1"
-AR Path="/57724D0D/577247BB" Ref="#PWR039"  Part="1"
-F 0 "#PWR039" H 1150 1400 50  0001 C CNN
+AR Path="/577246EF/577247BB" Ref="#PWR18"  Part="1"
+AR Path="/57724CA7/577247BB" Ref="#PWR26"  Part="1"
+AR Path="/57724D0D/577247BB" Ref="#PWR34"  Part="1"
+F 0 "#PWR18" H 1150 1400 50  0001 C CNN
 F 1 "+12V" H 1150 1690 50  0000 C CNN
 F 2 "" H 1150 1550 50  0000 C CNN
@@
 AR Path="/57724CA7/577247C1" Ref="U2"  Part="1"
 AR Path="/57724D0D/577247C1" Ref="U3"  Part="1"
-F 0 "U3" H 1250 2100 50  0001 L CNN
+F 0 "U1" H 1250 2100 50  0001 L CNN
 F 1 "LM311N" H 1250 2000 50  0000 L CNN
 F 2 "agg:MSOP-8" H 1250 1850 50  0001 C CNN
@@
 Wire Wire Line
 	950  1950 950  2450
-Wire Wire Line
-	950  2450 2650 2450
 Wire Wire Line
 	2650 2450 2650 1750
@@
 Text HLabel 950  1750 0    60   Input ~ 0
 VREF
+$Comp
+L GNDPWR #PWR25
+U 1 1 57728F8C
+P 2450 2050
+AR Path="/577246EF/57728F8C" Ref="#PWR25"  Part="1"
+AR Path="/57724CA7/57728F8C" Ref="#PWR33"  Part="1"
+AR Path="/57724D0D/57728F8C" Ref="#PWR41"  Part="1"
+F 0 "#PWR25" H 2450 1850 50  0001 C CNN
+F 1 "GNDPWR" H 2450 1900 50  0000 C CNN
+F 2 "" H 2450 2000 50  0000 C CNN
+F 3 "" H 2450 2000 50  0000 C CNN
+	1    2450 2050
+	1    0    0    -1
+$EndComp
+$Comp
+L VPP #PWR24
+U 1 1 57728FB5
+P 2450 950
+AR Path="/577246EF/57728FB5" Ref="#PWR24"  Part="1"
+AR Path="/57724CA7/57728FB5" Ref="#PWR32"  Part="1"
+AR Path="/57724D0D/57728FB5" Ref="#PWR40"  Part="1"
+F 0 "#PWR24" H 2450 800 50  0001 C CNN
+F 1 "VPP" H 2465 1123 50  0000 C CNN
+F 2 "" H 2450 950 50  0000 C CNN
+F 3 "" H 2450 950 50  0000 C CNN
+	1    2450 950
+	1    0    0    -1
+$EndComp
+Wire Wire Line
+	950  2450 2650 2450
 $EndSCHEMATC
