File: day-star.sch (KiCad schematic (older format))
At the start: 10 parts, among them Q1 Q_NMOS_DGS, Q2 Q_PMOS_DGS, U1 MCP6001

Commit message: Power pin wrangling
Parts:
- added P1: PWR_CONN, symbol CONN_01X02
Connections:
- wire segments 10 -> 12
Changed lines of the file:
@@
 L +36V #PWR01
 U 1 1 570F9388
-P 1800 1250
-F 0 "#PWR01" H 1800 1100 50  0001 C CNN
-F 1 "+36V" H 1800 1390 50  0000 C CNN
-F 2 "" H 1800 1250 50  0000 C CNN
-F 3 "" H 1800 1250 50  0000 C CNN
-	1    1800 1250
-	1    0    0    -1
+P 1050 800
+F 0 "#PWR01" H 1050 650 50  0001 C CNN
+F 1 "+36V" H 1050 940 50  0000 C CNN
+F 2 "" H 1050 800 50  0000 C CNN
+F 3 "" H 1050 800 50  0000 C CNN
+	1    1050 800
+	-1   0    0    -1
 $EndComp
 $Comp
@@
 L GND #PWR02
 U 1 1 570F9738
-P 2100 2450
-F 0 "#PWR02" H 2100 2200 50  0001 C CNN
-F 1 "GND" H 2100 2300 50  0000 C CNN
-F 2 "" H 2100 2450 50  0000 C CNN
-F 3 "" H 2100 2450 50  0000 C CNN
-	1    2100 2450
+P 1050 1000
+F 0 "#PWR02" H 1050 750 50  0001 C CNN
+F 1 "GND" H 1050 850 50  0000 C CNN
+F 2 "" H 1050 1000 50  0000 C CNN
+F 3 "" H 1050 1000 50  0000 C CNN
+	1    1050 1000
 	1    0    0    -1
 $EndComp
@@
 L PWR_FLAG #FLG07
 U 1 1 570FA127
-P 1800 1250
-F 0 "#FLG07" H 1800 1345 50  0001 C CNN
-F 1 "PWR_FLAG" H 1800 1430 50  0000 C CNN
-F 2 "" H 1800 1250 50  0000 C CNN
-F 3 "" H 1800 1250 50  0000 C CNN
-	1    1800 1250
-	0    -1   -1   0
+P 1050 800
+F 0 "#FLG07" H 1050 895 50  0001 C CNN
+F 1 "PWR_FLAG" V 1050 1150 50  0000 C CNN
+F 2 "" H 1050 800 50  0000 C CNN
+F 3 "" H 1050 800 50  0000 C CNN
+	1    1050 800
+	0    1    -1   0
 $EndComp
 $Comp
@@
 Text Label 3850 3100 2    60   ~ 0
 VREF
+Wire Wire Line
+	1050 850  1050 800
+Connection ~ 3300 1800
+$Comp
+L CONN_01X02 P1
+U 1 1 570FA4FC
+P 850 900
+F 0 "P1" H 850 1050 50  0001 C CNN
+F 1 "PWR_CONN" V 950 900 50  0000 C CNN
+F 2 "" H 850 900 50  0000 C CNN
+F 3 "" H 850 900 50  0000 C CNN
+	1    850  900
+	-1   0    0    -1
+$EndComp
+Connection ~ 1050 800
+$Comp
+L PWR_FLAG #FLG010
+U 1 1 570FA5A1
+P 1050 1000
+F 0 "#FLG010" H 1050 1095 50  0001 C CNN
+F 1 "PWR_FLAG" V 1050 1350 50  0000 C CNN
+F 2 "" H 1050 1000 50  0000 C CNN
+F 3 "" H 1050 1000 50  0000 C CNN
+	1    1050 1000
+	0    1    -1   0
+$EndComp
+Connection ~ 1050 1000
+Wire Wire Line
+	1050 950  1050 1000
+$Comp
+L +36V #PWR011
+U 1 1 570FA5C8
+P 1800 1250
+F 0 "#PWR011" H 1800 1100 50  0001 C CNN
+F 1 "+36V" H 1800 1390 50  0000 C CNN
+F 2 "" H 1800 1250 50  0000 C CNN
+F 3 "" H 1800 1250 50  0000 C CNN
+	1    1800 1250
+	-1   0    0    -1
+$EndComp
+$Comp
+L GND #PWR012
+U 1 1 570FA5D7
+P 2100 2450
+F 0 "#PWR012" H 2100 2200 50  0001 C CNN
+F 1 "GND" H 2100 2300 50  0000 C CNN
+F 2 "" H 2100 2450 50  0000 C CNN
+F 3 "" H 2100 2450 50  0000 C CNN
+	1    2100 2450
+	1    0    0    -1
+$EndComp
+Connection ~ 4050 2900
 $EndSCHEMATC

Commit message: 12V regulator and proper ref voltage creation.
Parts:
- added R6: 11K, symbol R
- added R7: 200R, symbol R
- added U2: LM7812, symbol LM7812
- RV1: value 1K -> 800R
Connections:
- net labels removed: +1V0

Commit message: Messing around
Parts:
- RV1: symbol POT -> POT-RESCUE-day-star
Changed lines of the file:
@@
 EESchema Schematic File Version 2
+LIBS:day-star-rescue
 LIBS:power
 LIBS:device
@@
 LIBS:contrib
 LIBS:valves
+LIBS:day-star-cache
 EELAYER 25 0
 EELAYER END
@@
 	1    0    0    -1
 $EndComp
-$Comp
-L GND #PWR04
-U 1 1 570F99D1
-P 4050 3500
-F 0 "#PWR04" H 4050 3250 50  0001 C CNN
-F 1 "GND" H 4050 3350 50  0000 C CNN
-F 2 "" H 4050 3500 50  0000 C CNN
-F 3 "" H 4050 3500 50  0000 C CNN
-	1    4050 3500
-	1    0    0    -1
-$EndComp
 Text Label 4600 3200 0    60   ~ 0
 CTRL
@@
 $EndComp
 $Comp
-L POT RV1
+L POT-RESCUE-day-star RV1
 U 1 1 570F9C63
 P 3800 1850
@@
 	1050 950  1050 1000
 $Comp
+L +12V #PWR010
+U 1 1 570FA767
+P 3800 1400
+F 0 "#PWR010" H 3800 1250 50  0001 C CNN
+F 1 "+12V" H 3800 1540 50  0000 C CNN
+F 2 "" H 3800 1400 50  0000 C CNN
+F 3 "" H 3800 1400 50  0000 C CNN
+	1    3800 1400
+	1    0    0    -1
+$EndComp
+$Comp
+L R R6
+U 1 1 570FA77B
+P 3800 1550
+F 0 "R6" V 3880 1550 50  0001 C CNN
+F 1 "11K" V 3800 1550 50  0000 C CNN
+F 2 "" V 3730 1550 50  0000 C CNN
+F 3 "" H 3800 1550 50  0000 C CNN
+	1    3800 1550
+	1    0    0    -1
+$EndComp
+$Comp
+L R R7
+U 1 1 570FA7ED
+P 3800 2150
+F 0 "R7" V 3880 2150 50  0001 C CNN
+F 1 "200R" V 3800 2150 50  0000 C CNN
+F 2 "" V 3730 2150 50  0000 C CNN
+F 3 "" H 3800 2150 50  0000 C CNN
+	1    3800 2150
+	1    0    0    -1
+$EndComp
+$Comp
+L LM7812 U2
+U 1 1 570FA94E
+P 2200 900
+F 0 "U2" H 2350 704 50  0001 C CNN
+F 1 "LM7812" H 2200 1100 50  0001 C CNN
+F 2 "" H 2200 900 50  0000 C CNN
+F 3 "" H 2200 900 50  0000 C CNN
+	1    2200 900
+	1    0    0    -1
+$EndComp
+$Comp
+L +36V #PWR011
+U 1 1 570FA9B1
+P 1800 850
+F 0 "#PWR011" H 1800 700 50  0001 C CNN
+F 1 "+36V" H 1800 990 50  0000 C CNN
+F 2 "" H 1800 850 50  0000 C CNN
+F 3 "" H 1800 850 50  0000 C CNN
+	1    1800 850
+	1    0    0    -1
+$EndComp
+$Comp
+L GND #PWR012
+U 1 1 570FA9C7
+P 2200 1150
+F 0 "#PWR012" H 2200 900 50  0001 C CNN
+F 1 "GND" H 2200 1000 50  0000 C CNN
+F 2 "" H 2200 1150 50  0000 C CNN
+F 3 "" H 2200 1150 50  0000 C CNN
+	1    2200 1150
+	1    0    0    -1
+$EndComp
+$Comp
+L GND #PWR09
+U 1 1 570FA5D7
+P 1750 3700
+F 0 "#PWR09" H 1750 3450 50  0001 C CNN
+F 1 "GND" H 1750 3550 50  0000 C CNN
+F 2 "" H 1750 3700 50  0000 C CNN
+F 3 "" H 1750 3700 50  0000 C CNN
+	1    1750 3700
+	1    0    0    -1
+$EndComp
+$Comp
+L GND #PWR04
+U 1 1 570F99D1
+P 4050 3500
+F 0 "#PWR04" H 4050 3250 50  0001 C CNN
+F 1 "GND" H 4050 3350 50  0000 C CNN
+F 2 "" H 4050 3500 50  0000 C CNN
+F 3 "" H 4050 3500 50  0000 C CNN
+	1    4050 3500
+	1    0    0    -1
+$EndComp
+$Comp
+L +12V #PWR013
+U 1 1 570FA9EE
+P 4050 2900
+F 0 "#PWR013" H 4050 2750 50  0001 C CNN
+F 1 "+12V" H 4050 3040 50  0000 C CNN
+F 2 "" H 4050 2900 50  0000 C CNN
+F 3 "" H 4050 2900 50  0000 C CNN
+	1    4050 2900
+	1    0    0    -1
+$EndComp
+$Comp
 L +36V #PWR08
 U 1 1 570FA5C8
@@
 	-1   0    0    -1
 $EndComp
-$Comp
-L GND #PWR09
-U 1 1 570FA5D7
-P 1750 3700
-F 0 "#PWR09" H 1750 3450 50  0001 C CNN
-F 1 "GND" H 1750 3550 50  0000 C CNN
-F 2 "" H 1750 3700 50  0000 C CNN
-F 3 "" H 1750 3700 50  0000 C CNN
-	1    1750 3700
-	1    0    0    -1
-$EndComp
-$Comp
-L +12V #PWR010
-U 1 1 570FA767
-P 3800 1400
-F 0 "#PWR010" H 3800 1250 50  0001 C CNN
-F 1 "+12V" H 3800 1540 50  0000 C CNN
-F 2 "" H 3800 1400 50  0000 C CNN
-F 3 "" H 3800 1400 50  0000 C CNN
-	1    3800 1400
-	1    0    0    -1
-$EndComp
-$Comp
-L R R6
-U 1 1 570FA77B
-P 3800 1550
-F 0 "R6" V 3880 1550 50  0001 C CNN
-F 1 "11K" V 3800 1550 50  0000 C CNN
-F 2 "" V 3730 1550 50  0000 C CNN
-F 3 "" H 3800 1550 50  0000 C CNN
-	1    3800 1550
-	1    0    0    -1
-$EndComp
-$Comp
-L R R7
-U 1 1 570FA7ED
-P 3800 2150
-F 0 "R7" V 3880 2150 50  0001 C CNN
-F 1 "200R" V 3800 2150 50  0000 C CNN
-F 2 "" V 3730 2150 50  0000 C CNN
-F 3 "" H 3800 2150 50  0000 C CNN
-	1    3800 2150
-	1    0    0    -1
-$EndComp
-$Comp
-L LM7812 U2
-U 1 1 570FA94E
-P 2200 900
-F 0 "U2" H 2350 704 50  0001 C CNN
-F 1 "LM7812" H 2200 1100 50  0001 C CNN
-F 2 "" H 2200 900 50  0000 C CNN
-F 3 "" H 2200 900 50  0000 C CNN
-	1    2200 900
-	1    0    0    -1
-$EndComp
-$Comp
-L +36V #PWR011
-U 1 1 570FA9B1
-P 1800 850
-F 0 "#PWR011" H 1800 700 50  0001 C CNN
-F 1 "+36V" H 1800 990 50  0000 C CNN
-F 2 "" H 1800 850 50  0000 C CNN
-F 3 "" H 1800 850 50  0000 C CNN
-	1    1800 850
-	1    0    0    -1
-$EndComp
-$Comp
-L GND #PWR012
-U 1 1 570FA9C7
-P 2200 1150
-F 0 "#PWR012" H 2200 900 50  0001 C CNN
-F 1 "GND" H 2200 1000 50  0000 C CNN
-F 2 "" H 2200 1150 50  0000 C CNN
-F 3 "" H 2200 1150 50  0000 C CNN
-	1    2200 1150
-	1    0    0    -1
-$EndComp
-$Comp
-L +12V #PWR013
-U 1 1 570FA9EE
-P 4050 2900
-F 0 "#PWR013" H 4050 2750 50  0001 C CNN
-F 1 "+12V" H 4050 3040 50  0000 C CNN
-F 2 "" H 4050 2900 50  0000 C CNN
-F 3 "" H 4050 2900 50  0000 C CNN
-	1    4050 2900
-	1    0    0    -1
-$EndComp
 $EndSCHEMATC

Commit message: Shiggles
Parts:
- removed D1: LED, symbol LED
- removed Q1: Q_NMOS_DGS, symbol Q_NMOS_DGS
- removed Q2: Q_PMOS_DGS, symbol Q_PMOS_DGS
- removed R3: 0R3, symbol R
- removed R4: 10K, symbol R
- removed R5: 82K, symbol R
- removed R7: 200R, symbol R
- removed U1: MCP6001, symbol MCP6001
- removed U2: LM7812, symbol LM7812
- added C1, C2: 100n, agg:0603, symbol C
- added C3: 1u, agg:0603, symbol C
- added PWR1: IFX21401, footprints:PG-SCT595-5, symbol IFX21401
- P1: footprint (none) -> agg:SIL-254P-02
- R1: value 10K -> 2k; footprint (none) -> agg:0603
- R2: value 22K -> 1k; footprint (none) -> agg:0603
- R3: renamed from R6; footprint (none) -> agg:0603
- RV1: value 800R -> 1k; footprint (none) -> agg:SIL-254P-03
Connections:
- net labels removed: CTRL, SENSE, VREF
- wire segments 12 -> 14

Commit message: Continuing shiggles
Parts:
- P1: footprint agg:SIL-254P-02 -> Terminal_Blocks:TerminalBlock_Pheonix_MKDS1.5-2pol
- R3: value 11K -> 11k9
- RV1: value 1k -> 100R
Changed lines of the file:
@@
 $EndDescr
 $Comp
-L +36V #PWR01
-U 1 1 570F9388
-P 1050 800
-F 0 "#PWR01" H 1050 650 50  0001 C CNN
-F 1 "+36V" H 1050 940 50  0000 C CNN
-F 2 "" H 1050 800 50  0000 C CNN
-F 3 "" H 1050 800 50  0000 C CNN
-	1    1050 800
-	-1   0    0    -1
-$EndComp
-$Comp
-L GND #PWR02
-U 1 1 570F9738
-P 1050 1000
-F 0 "#PWR02" H 1050 750 50  0001 C CNN
-F 1 "GND" H 1050 850 50  0000 C CNN
-F 2 "" H 1050 1000 50  0000 C CNN
-F 3 "" H 1050 1000 50  0000 C CNN
-	1    1050 1000
-	1    0    0    -1
-$EndComp
-$Comp
-L +12V #PWR03
+L +12V #PWR16
 U 1 1 570F99AF
 P 5000 1300
-F 0 "#PWR03" H 5000 1150 50  0001 C CNN
+F 0 "#PWR16" H 5000 1150 50  0001 C CNN
 F 1 "+12V" H 5000 1440 50  0000 C CNN
 F 2 "" H 5000 1300 50  0000 C CNN
@@
 $EndComp
 $Comp
-L GND #PWR04
+L GND #PWR2
 U 1 1 570F9C3D
 P 950 2700
-F 0 "#PWR04" H 950 2450 50  0001 C CNN
+F 0 "#PWR2" H 950 2450 50  0001 C CNN
 F 1 "GND" H 950 2550 50  0000 C CNN
 F 2 "" H 950 2700 50  0000 C CNN
@@
 P 950 2550
 F 0 "RV1" H 950 2470 50  0001 C CNN
-F 1 "1k" H 950 2550 50  0000 C CNN
+F 1 "100R" H 950 2550 50  0000 C CNN
 F 2 "agg:SIL-254P-03" H 950 2550 50  0001 C CNN
 F 3 "" H 950 2550 50  0000 C CNN
@@
 $EndComp
 $Comp
-L PWR_FLAG #FLG05
+L PWR_FLAG #FLG1
 U 1 1 570FA127
 P 1050 800
-F 0 "#FLG05" H 1050 895 50  0001 C CNN
+F 0 "#FLG1" H 1050 895 50  0001 C CNN
 F 1 "PWR_FLAG" V 1050 1150 50  0000 C CNN
 F 2 "" H 1050 800 50  0000 C CNN
@@
 	0    1    -1   0
 $EndComp
-Wire Wire Line
-	1050 850  1050 800
 $Comp
 L CONN_01X02 P1
@@
 F 0 "P1" H 850 1050 50  0001 C CNN
 F 1 "PWR_CONN" V 950 900 50  0000 C CNN
-F 2 "agg:SIL-254P-02" H 850 900 50  0001 C CNN
+F 2 "Terminal_Blocks:TerminalBlock_Pheonix_MKDS1.5-2pol" H 850 900 50  0001 C CNN
 F 3 "" H 850 900 50  0000 C CNN
 	1    850  900
 	-1   0    0    -1
 $EndComp
-Connection ~ 1050 800
-$Comp
-L PWR_FLAG #FLG06
+$Comp
+L PWR_FLAG #FLG2
 U 1 1 570FA5A1
 P 1050 1000
-F 0 "#FLG06" H 1050 1095 50  0001 C CNN
+F 0 "#FLG2" H 1050 1095 50  0001 C CNN
 F 1 "PWR_FLAG" V 1050 1350 50  0000 C CNN
 F 2 "" H 1050 1000 50  0000 C CNN
@@
 	0    1    -1   0
 $EndComp
-Connection ~ 1050 1000
-Wire Wire Line
-	1050 950  1050 1000
-$Comp
-L +12V #PWR07
+$Comp
+L +12V #PWR1
 U 1 1 570FA767
 P 950 2100
-F 0 "#PWR07" H 950 1950 50  0001 C CNN
+F 0 "#PWR1" H 950 1950 50  0001 C CNN
 F 1 "+12V" H 950 2240 50  0000 C CNN
 F 2 "" H 950 2100 50  0000 C CNN
@@
 P 950 2250
 F 0 "R3" V 1030 2250 50  0001 C CNN
-F 1 "11K" V 950 2250 50  0000 C CNN
+F 1 "11k9" V 950 2250 50  0000 C CNN
 F 2 "agg:0603" V 880 2250 50  0001 C CNN
 F 3 "" H 950 2250 50  0000 C CNN
@@
 $EndComp
 $Comp
-L +36V #PWR08
+L +36V #PWR12
 U 1 1 570FA9B1
 P 3500 1300
-F 0 "#PWR08" H 3500 1150 50  0001 C CNN
+F 0 "#PWR12" H 3500 1150 50  0001 C CNN
 F 1 "+36V" H 3500 1440 50  0000 C CNN
 F 2 "" H 3500 1300 50  0000 C CNN
@@
 $EndComp
 $Comp
-L GND #PWR09
+L GND #PWR15
 U 1 1 570FA9C7
 P 4800 1350
-F 0 "#PWR09" H 4800 1100 50  0001 C CNN
+F 0 "#PWR15" H 4800 1100 50  0001 C CNN
 F 1 "GND" H 4800 1200 50  0000 C CNN
 F 2 "" H 4800 1350 50  0000 C CNN
@@
 F2 "VREF" I L 1950 3050 60
 $EndSheet
-Wire Wire Line
-	1950 2050 1750 2050
-Wire Wire Line
-	1750 2050 1750 2550
-Wire Wire Line
-	1100 2550 1950 2550
-Wire Wire Line
-	1950 3050 1600 3050
-Wire Wire Line
-	1600 3050 1600 2550
-Connection ~ 1750 2550
-Connection ~ 1600 2550
 $Comp
 L IFX21401 PWR1
@@
 	1    0    0    -1
 $EndComp
-Wire Wire Line
-	4750 1300 5000 1300
-Wire Wire Line
-	4750 1150 4800 1150
-$Comp
-L GND #PWR010
+$Comp
+L GND #PWR14
 U 1 1 57726027
 P 3700 1350
-F 0 "#PWR010" H 3700 1100 50  0001 C CNN
+F 0 "#PWR14" H 3700 1100 50  0001 C CNN
 F 1 "GND" H 3700 1200 50  0000 C CNN
 F 2 "" H 3700 1350 50  0000 C CNN
@@
 	1    0    0    -1
 $EndComp
-Wire Wire Line
-	3750 1200 3700 1200
-Wire Wire Line
-	3500 1300 3750 1300
-Wire Wire Line
-	3700 1200 3700 1350
-Wire Wire Line
-	4800 1150 4800 1350
 $Comp
 L R R1
@@
 $EndComp
 $Comp
-L +36V #PWR011
+L +36V #PWR9
 U 1 1 57726469
 P 2800 800
-F 0 "#PWR011" H 2800 650 50  0001 C CNN
+F 0 "#PWR9" H 2800 650 50  0001 C CNN
 F 1 "+36V" H 2800 940 50  0000 C CNN
 F 2 "" H 2800 800 50  0000 C CNN
@@
 $EndComp
 $Comp
-L GND #PWR012
+L GND #PWR10
 U 1 1 57726489
 P 2800 1400
-F 0 "#PWR012" H 2800 1150 50  0001 C CNN
+F 0 "#PWR10" H 2800 1150 50  0001 C CNN
 F 1 "GND" H 2800 1250 50  0000 C CNN
 F 2 "" H 2800 1400 50  0000 C CNN
@@
 	1    0    0    -1
 $EndComp
-Wire Wire Line
-	2800 1100 3750 1100
-Connection ~ 2800 1100
 $Comp
 L C C3
@@
 	1    0    0    -1
 $EndComp
-Connection ~ 5000 1300
-$Comp
-L GND #PWR013
+$Comp
+L GND #PWR17
 U 1 1 577266CD
 P 5000 1600
-F 0 "#PWR013" H 5000 1350 50  0001 C CNN
+F 0 "#PWR17" H 5000 1350 50  0001 C CNN
 F 1 "GND" H 5000 1450 50  0000 C CNN
 F 2 "" H 5000 1600 50  0000 C CNN
@@
 	1    0    0    -1
 $EndComp
-Connection ~ 3500 1300
-$Comp
-L GND #PWR014
+$Comp
+L GND #PWR13
 U 1 1 57726884
 P 3500 1600
-F 0 "#PWR014" H 3500 1350 50  0001 C CNN
+F 0 "#PWR13" H 3500 1350 50  0001 C CNN
 F 1 "GND" H 3500 1450 50  0000 C CNN
 F 2 "" H 3500 1600 50  0000 C CNN
@@
 $EndComp
 $Comp
-L GND #PWR015
+L GND #PWR11
 U 1 1 577268C5
 P 3150 1400
-F 0 "#PWR015" H 3150 1150 50  0001 C CNN
+F 0 "#PWR11" H 3150 1150 50  0001 C CNN
 F 1 "GND" H 3150 1250 50  0000 C CNN
 F 2 "" H 3150 1400 50  0000 C CNN
@@
 	1    0    0    -1
 $EndComp
+$Comp
+L VPP #PWR3
+U 1 1 577292AD
+P 1050 800
+F 0 "#PWR3" H 1050 650 50  0001 C CNN
+F 1 "VPP" H 1065 973 50  0000 C CNN
+F 2 "" H 1050 800 50  0000 C CNN
+F 3 "" H 1050 800 50  0000 C CNN
+	1    1050 800
+	1    0    0    -1
+$EndComp
+$Comp
+L GNDPWR #PWR4
+U 1 1 577292D5
+P 1050 1000
+F 0 "#PWR4" H 1050 800 50  0001 C CNN
+F 1 "GNDPWR" H 1050 850 50  0000 C CNN
+F 2 "" H 1050 950 50  0000 C CNN
+F 3 "" H 1050 950 50  0000 C CNN
+	1    1050 1000
+	1    0    0    -1
+$EndComp
+$Comp
+L VPP #PWR5
+U 1 1 5772931B
+P 1850 1200
+F 0 "#PWR5" H 1850 1050 50  0001 C CNN
+F 1 "VPP" H 1865 1373 50  0000 C CNN
+F 2 "" H 1850 1200 50  0000 C CNN
+F 3 "" H 1850 1200 50  0000 C CNN
+	1    1850 1200
+	1    0    0    -1
+$EndComp
+$Comp
+L GNDPWR #PWR6
+U 1 1 5772933C
+P 1850 1300
+F 0 "#PWR6" H 1850 1100 50  0001 C CNN
+F 1 "GNDPWR" H 1850 1150 50  0000 C CNN
+F 2 "" H 1850 1250 50  0000 C CNN
+F 3 "" H 1850 1250 50  0000 C CNN
+	1    1850 1300
+	1    0    0    -1
+$EndComp
+$Comp
+L +36V #PWR7
+U 1 1 5772935C
+P 2250 1200
+F 0 "#PWR7" H 2250 1050 50  0001 C CNN
+F 1 "+36V" H 2250 1340 50  0000 C CNN
+F 2 "" H 2250 1200 50  0000 C CNN
+F 3 "" H 2250 1200 50  0000 C CNN
+	1    2250 1200
+	1    0    0    -1
+$EndComp
+$Comp
+L GND #PWR8
+U 1 1 5772937C
+P 2250 1300
+F 0 "#PWR8" H 2250 1050 50  0001 C CNN
+F 1 "GND" H 2250 1150 50  0000 C CNN
+F 2 "" H 2250 1300 50  0000 C CNN
+F 3 "" H 2250 1300 50  0000 C CNN
+	1    2250 1300
+	1    0    0    -1
+$EndComp
 Connection ~ 3150 1100
+Connection ~ 3500 1300
+Connection ~ 5000 1300
+Connection ~ 2800 1100
+Wire Wire Line
+	2800 1100 3750 1100
+Wire Wire Line
+	4800 1150 4800 1350
+Wire Wire Line
+	3700 1200 3700 1350
+Wire Wire Line
+	3500 1300 3750 1300
+Wire Wire Line
+	3750 1200 3700 1200
+Wire Wire Line
+	4750 1150 4800 1150
+Wire Wire Line
+	4750 1300 5000 1300
+Connection ~ 1600 2550
+Connection ~ 1750 2550
+Wire Wire Line
+	1600 3050 1600 2550
+Wire Wire Line
+	1950 3050 1600 3050
+Wire Wire Line
+	1100 2550 1950 2550
+Wire Wire Line
+	1750 2050 1750 2550
+Wire Wire Line
+	1950 2050 1750 2050
+Wire Wire Line
+	1050 950  1050 1000
+Connection ~ 1050 1000
+Connection ~ 1050 800
+Wire Wire Line
+	1050 850  1050 800
+Wire Wire Line
+	1850 1200 2250 1200
+Wire Wire Line
+	2250 1300 1850 1300
 $EndSCHEMATC

Commit message: Tweaked bits and started setup for IC driven version
Parts:
- removed C1, C2: 100n, agg:0603, symbol C
- removed C3: 1u, agg:0603, symbol C
- removed PWR1: IFX21401, footprints:PG-SCT595-5, symbol IFX21401
- removed R1: 2k, agg:0603, symbol R
- removed R2: 1k, agg:0603, symbol R
- removed R3: 11k9, agg:0603, symbol R
- removed RV1: 100R, agg:SIL-254P-03, symbol POT-RESCUE-day-star
- added IC? (x3): TPS92512, agg:MSOP-10-EP-TI, symbol TPS92512
- added IC?: STM32F0xxKxTx, agg:LQFP-32, symbol STM32F0xxKxTx
- added P?: LEDA, symbol CONN_01X02
- added P?: LEDB, symbol CONN_01X02
- added P?: LEDC, symbol CONN_01X02
- added U?: ESP8266-ESP01, agg-unchecked:ESP01, symbol ESP8266-ESP01
Connections:
- net +36V renamed +48V

Commit message: More shenanigans, starting to put together power supplies
Parts:
- removed IC? (x2): TPS92512, agg:MSOP-10-EP-TI, symbol TPS92512
- removed P?: LEDB, symbol CONN_01X02
- removed P?: LEDC, symbol CONN_01X02
- removed U?: ESP8266-ESP01, agg-unchecked:ESP01, symbol ESP8266-ESP01
- added C? (x9): C, symbol C_Small
- added D?: D, symbol D_Schottky_Small
- added L? (x2): L, symbol INDUCTOR_Small
- added P?: SWD_TC, agg:TC2030-NL, symbol SWD_TC
- added P?: FTDI_CONN, Pin_Headers:Pin_Header_Angled_2x06, symbol FTDI_CONN
- added R? (x6): R, symbol R_Small
- added RV?: POT, symbol POT
- added U?: ESP-12E, symbol ESP-12E
- added U?: MAX17501, symbol MAX17501
Connections:
- net +48V: now also IC?.2 (VIN), C?.2, C?.2, R?.2, R?.2, U?.2 (VIN), U?.3 (EN/UVLO)
- net GND: now also IC?.9 (GND), IC?.EP (GND), C?.1, C?.1, C?.1, C?.1, C?.1, C?.1, C?.1, D?.2 (A), R?.1, R?.1, R?.1, U?.1 (PGND), U?.9 (GND), U?.EP
- net at IC?.1 (BOOT): now also C?.2
- net at IC?.10 (PH): now also C?.1, D?.1 (K), L?.2
- net at IC?.3 (UVLO): now also R?.1, R?.2
- net DIM: now reaches IC?.4 (PDIM)
- net at IC?.5 (RT/CLK): now also R?.2
- net at IC?.6 (IADJ): now also C?.2, R?.1
- net at IC?.7 (ISENSE): now also R?.2
- net at IC?.8 (COMP): now also C?.2
- net at P?.1 (P1): now also C?.2, L?.1
- net at P?.2 (P2): now also C?.1, R?.1, R?.2
- new net: L?.2, U?.10 (LX)
- new net: C?.2, U?.4 (VCC)
- new net: C?.2, U?.6 (SS)
- new net +3V3: C?.2, L?.1, U?.5 (FB/VO)
- no-connect marks 0 -> 1
Other:
- moved on the sheet: IC?, P?

Commit message: More schematic wrangling
Parts:
- added C? (x12): C, symbol C_Small
- added C?: 0u1, symbol C_Small
- added C? (x2): 100n, symbol C_Small
- added C?: 4u7, symbol C_Small
- added C?: 10n, symbol C_Small
- added C?: 1u, symbol C_Small
- added D? (x2): D, symbol D_Schottky_Small
- added IC? (x2): TPS92512, agg:MSOP-10-EP-TI, symbol TPS92512
- added L? (x2): L, symbol INDUCTOR_Small
- added P? (x2): LEDA, symbol CONN_01X02
- added R? (x16): R, symbol R_Small
Connections:
- net +3V3: now also IC?.1 (VDD), IC?.17 (VDD), IC?.5 (VDDA), P?.1 (VDD), RV?.1, U?.8 (VCC), C?.2, C?.2, C?.2, C?.2, C?.2, C?.2, C?.2
- net +48V: now also C?.2, C?.2, IC?.2 (VIN), IC?.2 (VIN), R?.2, R?.2, R?.2, R?.2
- net GND: now also IC?.16 (VSS), IC?.32 (VSS), P?.11 (GND), P?.5 (GND), RV?.3, U?.15 (GND), C?.1, C?.1, C?.1, C?.1, C?.1, C?.1, C?.1, C?.1, C?.1, C?.1, C?.1, C?.1, C?.1, C?.1, D?.2 (A), D?.2 (A), IC?.9 (GND), IC?.9 (GND), IC?.EP (GND), IC?.EP (GND), R?.1, R?.1, R?.1, R?.1, R?.1, R?.1, R?.1
- net SWDIO: now reaches IC?.23 (PA13)
- net SWDIO: now also P?.2 (SWDIO)
- net SWCLK: now reaches IC?.24 (PA14)
- net SWCLK: now also P?.4 (SWDCLK)
- net STMRST: now reaches IC?.4 (NRST)
- net STMRST: now also P?.3 (~RST), C?.2
- net ANDIM: now reaches RV?.2
- net FTDIRTS: now reaches U?.1 (RST)
- net FTDIRTS: now also P?.1 (RTS)
- net FTDIDTR: now reaches U?.18 (GPIO0)
- net FTDIDTR: now also P?.4 (DTR)
- net ESPRX: now reaches U?.21 (RXD0)
- net ESPRX: now also R?.1
- net ESPTX: now reaches U?.22 (TXD0)
- net ESPTX: now also R?.1
- net ESPEN: now reaches U?.3 (CH_PD)
- net ESPEN: now also R?.2
- net at P?.3 (RXD): now also R?.2
- net at P?.5 (TXD): now also R?.2
- net at P?.7 (VCC): now also R?.2
- net DIM renamed PWMDIM
- net PWMDIM: now also IC?.4 (PDIM), IC?.4 (PDIM)
- new net: C?.2, IC?.1 (BOOT) (x2)
- new net: C?.1, D?.1 (K), IC?.10 (PH), L?.2 (x2)
- new net: IC?.3 (UVLO), R?.1, R?.2 (x2)
- new net: IC?.5 (RT/CLK), R?.2 (x2)
- new net: C?.2, IC?.6 (IADJ), R?.1 (x2)
- new net: IC?.7 (ISENSE), R?.2 (x2)
- new net: C?.2, IC?.8 (COMP) (x2)
- new net: C?.2, L?.1, P?.1 (P1) (x2)
- new net: C?.1, P?.2 (P2), R?.1, R?.2 (x2)
- new net FTDIVCC: R?.1
- no-connect marks 1 -> 21
Other:
- note added: "VDD DECOUPLE"
- note added: "VDDA DECOUPLE"
- moved on the sheet: IC?, P?, RV?, U?
