File: day-star.sch (KiCad schematic (older format))
At the start: 69 parts, among them P1 PWR_CONN

Commit message: Bunch of small changes
Parts:
- removed C? (x10): C, symbol C_Small
- removed D? (x2): D, symbol D_Schottky_Small
- removed IC? (x2): TPS92512, agg:MSOP-10-EP-TI, symbol TPS92512
- removed L? (x2): L, symbol INDUCTOR_Small
- removed P? (x2): LEDA, symbol CONN_01X02
- removed R? (x14): R, symbol R_Small
- removed RV?: POT, symbol POT
- added R? (x2): 3k3, symbol R_Small
- added R?: 100k, symbol R_Small
- added U?: POT_SW, symbol POT_SW
- C?: value C -> 100n
- C?: value C -> 22u
- R?: value R -> 100k
- R?: value R -> 3k3
Connections:
- net +3V3: now also U?.1, U?.5
- net ANDIM: now also U?.2
- net ESPRX: now also R?.1
- net FTDIVCC: now also R?.1
- net GND: now also R?.1, U?.3
- net at P?.5 (TXD): now also R?.2
- net at P?.7 (VCC): now also R?.2
- new net ONOFFSW: R?.2, U?.4
