File: controller/day-star.sch (KiCad schematic (older format))
At the start: 33 parts, among them IC1 STM32F0xxKxTx, P1 PWR_CONN, P2 LEDA, P3 LEDB, P4 LEDC, P6 FTDI_CONN, U1 ESP-12E

Commit message: More controller tweaks
Parts:
- added C?: 2u2, symbol C_Small
- added C?: 22u, symbol C_Small
- added L?: 10u, symbol INDUCTOR_Small
- added R?: 100k, symbol R_Small
Connections:
- net +12V: now also U?.2 (VIN), U?.3 (EN), C?.2
- net +3V3: now also U?.10 (VOS), C?.2, L?.1, R?.2
- net GND: now also U?.1 (PGND), U?.11 (ETP), U?.4 (NC), U?.5 (FB), U?.6 (AGND), C?.1, C?.1
- net at U?.7 (PG): now also R?.1
- net at U?.9 (SW): now also L?.2
Changed lines of the file:
@@
+	1    0    0    -1
+$EndComp
+$Comp
+L GND #PWR?
+U 1 1 5851451D
+P 4200 3450
+F 0 "#PWR?" H 4200 3200 50  0001 C CNN
+F 1 "GND" H 4205 3277 50  0000 C CNN
+F 2 "" H 4200 3450 50  0000 C CNN
+F 3 "" H 4200 3450 50  0000 C CNN
+	1    4200 3450
+	1    0    0    -1
+$EndComp
+Wire Wire Line
+	4200 3450 4200 3350
+Connection ~ 4200 3450
+$Comp
+L GND #PWR?
+U 1 1 585145C6
+P 3700 3750
+F 0 "#PWR?" H 3700 3500 50  0001 C CNN
+F 1 "GND" H 3705 3577 50  0000 C CNN
+F 2 "" H 3700 3750 50  0000 C CNN
+F 3 "" H 3700 3750 50  0000 C CNN
+	1    3700 3750
+	1    0    0    -1
+$EndComp
+$Comp
+L GND #PWR?
+U 1 1 58514634
+P 2875 3450
+F 0 "#PWR?" H 2875 3200 50  0001 C CNN
+F 1 "GND" H 2880 3277 50  0000 C CNN
+F 2 "" H 2875 3450 50  0000 C CNN
+F 3 "" H 2875 3450 50  0000 C CNN
+	1    2875 3450
+	1    0    0    -1
+$EndComp
+Wire Wire Line
+	3200 3350 3200 3450
+Connection ~ 3200 3450
+$Comp
+L +12V #PWR?
+U 1 1 5851474E
+P 2875 3050
+F 0 "#PWR?" H 2875 2900 50  0001 C CNN
+F 1 "+12V" H 2890 3223 50  0000 C CNN
+F 2 "" H 2875 3050 50  0000 C CNN
+F 3 "" H 2875 3050 50  0000 C CNN
+	1    2875 3050
+	1    0    0    -1
+$EndComp
+$Comp
+L C_Small C?
+U 1 1 58514804
+P 2875 3250
+F 0 "C?" V 2646 3250 50  0001 C CNN
+F 1 "2u2" H 3025 3325 50  0000 R CNN
+F 2 "" H 2875 3250 50  0000 C CNN
+F 3 "" H 2875 3250 50  0000 C CNN
+	1    2875 3250
+	-1   0    0    1
+$EndComp
+Wire Wire Line
+	2875 3050 3200 3050
+Wire Wire Line
+	3200 3050 3200 3150
+Connection ~ 3200 3050
+Wire Wire Line
+	3200 3450 2875 3450
+Wire Wire Line
+	2875 3050 2875 3150
+Connection ~ 2875 3050
+Wire Wire Line
+	2875 3450 2875 3350
+Connection ~ 2875 3450
+$Comp
+L INDUCTOR_Small L?
+U 1 1 58514C74
+P 4300 3050
+F 0 "L?" V 4122 3050 50  0001 C CNN
+F 1 "10u" V 4250 3050 50  0000 C CNN
+F 2 "" H 4300 3050 50  0000 C CNN
+F 3 "" H 4300 3050 50  0000 C CNN
+	1    4300 3050
+	0    1    1    0
+$EndComp
+$Comp
+L R_Small R?
+U 1 1 58514CBE
+P 4500 3150
+F 0 "R?" H 4559 3196 50  0001 L CNN
+F 1 "100k" H 4450 3150 50  0000 R CNN
+F 2 "" H 4500 3150 50  0000 C CNN
+F 3 "" H 4500 3150 50  0000 C CNN
+	1    4500 3150
+	-1   0    0    1
+$EndComp
+$Comp
+L C_Small C?
+U 1 1 58514CE4
+P 4800 3250
+F 0 "C?" V 4571 3250 50  0001 C CNN
+F 1 "22u" H 4700 3250 50  0000 R CNN
+F 2 "" H 4800 3250 50  0000 C CNN
+F 3 "" H 4800 3250 50  0000 C CNN
+	1    4800 3250
+	-1   0    0    1
+$EndComp
+Wire Wire Line
+	4200 3150 4450 3150
+Wire Wire Line
+	4450 3150 4450 3050
+Wire Wire Line
+	4400 3050 4800 3050
+Connection ~ 4450 3050
+Wire Wire Line
+	4200 3250 4500 3250
+Wire Wire Line
+	4800 3050 4800 3150
+Connection ~ 4500 3050
+Wire Wire Line
+	4800 3350 4800 3450
+Wire Wire Line
+	4800 3450 4200 3450
+$Comp
+L +3V3 #PWR?
+U 1 1 58515113
+P 4800 3050
+F 0 "#PWR?" H 4800 2900 50  0001 C CNN
+F 1 "+3V3" H 4815 3223 50  0000 C CNN
+F 2 "" H 4800 3050 50  0000 C CNN
+F 3 "" H 4800 3050 50  0000 C CNN
+	1    4800 3050
 	1    0    0    -1
 $EndComp
